File: KiCAD/8-Bit CPU 32k.sch (KiCad schematic (older format))
At the start: 15 parts, among them J1 UART, SW1 RESET, U1 74HC04, X1 ACO-1.8432MHz

Commit message: Revision 1.2
Other:
- moved on the sheet: R9, SW1
Changed lines of the file:
@@
 Sheet 1 9
 Title "Minimal UART Computer"
-Date "2020-12-14"
+Date "2020-12-16"
 Rev "1.2"
 Comp ""
@@
 U 1 1 5F351101
 P 1150 2400
-F 0 "J1" H 1050 2750 50  0000 C CNN
-F 1 "UART" H 1050 2000 50  0000 C CNN
+F 0 "J1" H 1050 2900 50  0000 C CNN
+F 1 "UART" H 1050 2750 50  0000 C CNN
 F 2 "Connector_PinSocket_2.54mm:PinSocket_1x06_P2.54mm_Vertical" H 1150 2400 50  0001 C CNN
 F 3 "~" H 1150 2400 50  0001 C CNN
@@
 L power:GND #PWR0124
 U 1 1 5FC2AC5B
-P 5000 2700
+P 1250 1400
 AR Path="/5FC2AC5B" Ref="#PWR0124"  Part="1"
 AR Path="/5EC57429/5FC2AC5B" Ref="#PWR?"  Part="1"
-F 0 "#PWR0124" H 5000 2450 50  0001 C CNN
-F 1 "GND" H 5005 2527 50  0000 C CNN
-F 2 "" H 5000 2700 50  0001 C CNN
-F 3 "" H 5000 2700 50  0001 C CNN
-	1    5000 2700
+F 0 "#PWR0124" H 1250 1150 50  0001 C CNN
+F 1 "GND" H 1255 1227 50  0000 C CNN
+F 2 "" H 1250 1400 50  0001 C CNN
+F 3 "" H 1250 1400 50  0001 C CNN
+	1    1250 1400
 	1    0    0    -1
 $EndComp
@@
 L Switch:SW_Push SW1
 U 1 1 5FC2AC61
-P 5200 2700
+P 1450 1400
 AR Path="/5FC2AC61" Ref="SW1"  Part="1"
 AR Path="/5EC57429/5FC2AC61" Ref="SW?"  Part="1"
-F 0 "SW1" H 5200 2985 50  0000 C CNN
-F 1 "RESET" H 5200 2894 50  0000 C CNN
-F 2 "Button_Switch_THT:SW_PUSH_6mm" H 5200 2900 50  0001 C CNN
-F 3 "~" H 5200 2900 50  0001 C CNN
-	1    5200 2700
+F 0 "SW1" H 1450 1685 50  0000 C CNN
+F 1 "RESET" H 1450 1594 50  0000 C CNN
+F 2 "Button_Switch_THT:SW_PUSH_6mm" H 1450 1600 50  0001 C CNN
+F 3 "~" H 1450 1600 50  0001 C CNN
+	1    1450 1400
 	1    0    0    -1
 $EndComp
@@
 L power:+5V #PWR0160
 U 1 1 5FC3CDAD
-P 5400 2400
+P 1650 1100
 AR Path="/5FC3CDAD" Ref="#PWR0160"  Part="1"
 AR Path="/5EC57429/5FC3CDAD" Ref="#PWR?"  Part="1"
-F 0 "#PWR0160" H 5400 2250 50  0001 C CNN
-F 1 "+5V" H 5415 2573 50  0000 C CNN
-F 2 "" H 5400 2400 50  0001 C CNN
-F 3 "" H 5400 2400 50  0001 C CNN
-	1    5400 2400
+F 0 "#PWR0160" H 1650 950 50  0001 C CNN
+F 1 "+5V" H 1665 1273 50  0000 C CNN
+F 2 "" H 1650 1100 50  0001 C CNN
+F 3 "" H 1650 1100 50  0001 C CNN
+	1    1650 1100
 	1    0    0    -1
 $EndComp
@@
 L Device:R R9
 U 1 1 5FC3CDB3
-P 5400 2550
+P 1650 1250
 AR Path="/5FC3CDB3" Ref="R9"  Part="1"
 AR Path="/5EC57429/5FC3CDB3" Ref="R?"  Part="1"
-F 0 "R9" H 5250 2500 50  0000 L CNN
-F 1 "10k" V 5400 2450 50  0000 L CNN
-F 2 "Resistor_THT:R_Axial_DIN0207_L6.3mm_D2.5mm_P7.62mm_Horizontal" V 5330 2550 50  0001 C CNN
-F 3 "~" H 5400 2550 50  0001 C CNN
-	1    5400 2550
+F 0 "R9" H 1500 1200 50  0000 L CNN
+F 1 "10k" V 1650 1150 50  0000 L CNN
+F 2 "Resistor_THT:R_Axial_DIN0207_L6.3mm_D2.5mm_P7.62mm_Horizontal" V 1580 1250 50  0001 C CNN
+F 3 "~" H 1650 1250 50  0001 C CNN
+	1    1650 1250
 	-1   0    0    1
 $EndComp
-Text GLabel 5550 2700 2    50   Output ~ 0
+Text GLabel 1800 1400 2    50   Output ~ 0
 ~Reset
 Wire Wire Line
-	5400 2700 5550 2700
-Connection ~ 5400 2700
+	1650 1400 1800 1400
+Connection ~ 1650 1400
 Text GLabel 2450 4350 0    50   Input ~ 0
 ~Reset
