File: KiCAD/8-Bit CPU 32k.kicad_pcb (KiCad board)
At the start: 2 copper layers, 191.8 x 121.3 mm, 109 parts, among them J1 UART, SW1 RESET, U1 74HC04, U10 74HC173, U11 74HC161, U12 74HC86, U13 74HC283, U14 74HC283, U15 74HC245, U16 74HC86, U17 74HC173, U18 74HC02, U19 74HC08, U2 74HC173, U23 74HC245, U24 74HC32, U26 74HC161, U28 74HC161, U29 74HC32, U3 74HC173, U30 74HC161, U31 AT28C64B 8k ROM, U32 CY62256 32k RAM, U33 74HC161, U34 74HC161, U35 74HC00, U36 74HC173, U37 74HC193, U38 74HC173, U39 74HC164, U4 74HC245, U40 74HC02, U41 74HC173, U42 74HC161, U43 74HC165, U44 74HC00, U45 74HC165, U46 74HC161, U48 74HC32, U49 74HC161, U5 74HC173, U50 74HC245, U51 74HC161, U52 74HC161, U53 74HC245, U6 74HC173, U7 AT28C64B CTRL MSB, U8 74HC173, U9 AT28C64B CTRL LSB, X1 ACO-1.8432MHz

Commit message: Revision 1.2
Parts:
- C10: value 22pF -> 47pF
- C52: value 47µ -> 47µF
- R10: value 50 -> wire

Commit message: Revision 1.2.0
Parts:
- C10: value 47pF -> 100pF
Other:
- board text added: "Designed by C. Herting (slu4) 2020"
- board text added: "unlabeled caps: 100nF"
- board text removed: "designed by slu4 (2020)"
Changed lines of the file:
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@@
   (general
     (thickness 1.6)
-    (drawings 13)
+    (drawings 14)
     (tracks 4364)
     (zones 0)
@@
       (effects (font (size 1 1) (thickness 0.15)))
     )
-    (fp_text value 47pF (at -3.175 0.635) (layer F.SilkS)
+    (fp_text value 100pF (at -3.81 0.635) (layer F.SilkS)
       (effects (font (size 1 1) (thickness 0.15)))
     )
@@
     )
   )
+  (gr_text "unlabeled caps: 100nF" (at 55.245 157.48) (layer F.SilkS)
+    (effects (font (size 1 1) (thickness 0.15)))
+  )
   (gr_text "UART configuration: 5V, 115200bps, 8 data bits, no parity bit, 1 stop bit, flow control: none, transmit delay: 20ms per line" (at 186.055 157.48) (layer F.SilkS)
     (effects (font (size 1 1) (thickness 0.15)))
@@
     (effects (font (size 1 1) (thickness 0.15)))
   )
-  (gr_text "designed by slu4 (2020)" (at 109.855 40.005) (layer F.SilkS)
+  (gr_text "Designed by C. Herting (slu4) 2020" (at 111.125 40.005) (layer F.SilkS)
     (effects (font (size 1 1) (thickness 0.15)))
   )
@@
     (effects (font (size 1 1) (thickness 0.15)))
   )
-  (gr_text "Minimal UART CPU 1.2" (at 62.23 40.64) (layer F.SilkS)
+  (gr_text "Minimal UART CPU 1.2" (at 62.865 40.64) (layer F.SilkS)
     (effects (font (size 2 2) (thickness 0.15)))
   )
