File: KiCAD/IR.sch (KiCad schematic (older format))
At the start: 16 parts, among them U1 74HC04, U11 74HC161, U19 74HC08, U5 74HC173, U6 74HC173, U7 AT28C64B CTRL MSB, U8 74HC173, U9 AT28C64B CTRL LSB

Commit message: Revision 1.2
Parts:
- C10: value 22pF -> 47pF
- R10: value 50 -> wire
Changed lines of the file:
@@
 Sheet 3 9
 Title "Control Logic"
-Date "2020-12-14"
+Date "2020-12-16"
 Rev "1.2"
-Comp "Carsten (Slu4) Herting (c) 2020"
+Comp "by Carsten Herting (2020)"
 Comment1 ""
 Comment2 "creativecommons.org/licenses/by-nc-sa/3.0/deed.en"
@@
 ~FI
 $Comp
-L Device:R R?
-U 1 1 5FC2A84D
-P 8150 2050
-AR Path="/5FC2A84D" Ref="R?"  Part="1"
-AR Path="/5EC57429/5FC2A84D" Ref="R10"  Part="1"
-F 0 "R10" H 7950 2050 50  0000 L CNN
-F 1 "50" V 8150 2000 50  0000 L CNN
-F 2 "Resistor_THT:R_Axial_DIN0207_L6.3mm_D2.5mm_P7.62mm_Horizontal" V 8080 2050 50  0001 C CNN
-F 3 "~" H 8150 2050 50  0001 C CNN
-	1    8150 2050
-	-1   0    0    1
-$EndComp
-$Comp
 L Device:C_Small C?
 U 1 1 5FC2AF22
@@
 AR Path="/5F645851/5FC2AF22" Ref="C?"  Part="1"
 AR Path="/5EC57429/5FC2AF22" Ref="C10"  Part="1"
-F 0 "C10" V 8200 1800 50  0000 L CNN
-F 1 "22pF" V 7950 1800 50  0000 L CNN
+F 0 "C10" V 7950 1600 50  0000 L CNN
+F 1 "47pF" V 7950 1800 50  0000 L CNN
 F 2 "Capacitor_THT:C_Disc_D5.0mm_W2.5mm_P2.50mm" H 8050 1900 50  0001 C CNN
 F 3 "~" H 8050 1900 50  0001 C CNN
@@
 	0    1    1    0
 $EndComp
-Connection ~ 8150 1900
 $Comp
 L power:GND #PWR?
@@
 	1    0    0    -1
 $EndComp
-Wire Wire Line
-	8150 3100 8150 2200
 Connection ~ 3100 2300
 Connection ~ 5200 2300
 Connection ~ 7400 2300
 Connection ~ 10050 2300
+Wire Wire Line
+	8150 3100 8150 2200
+Connection ~ 8150 1900
+$Comp
+L Device:R R?
+U 1 1 5FC2A84D
+P 8150 2050
+AR Path="/5FC2A84D" Ref="R?"  Part="1"
+AR Path="/5EC57429/5FC2A84D" Ref="R10"  Part="1"
+F 0 "R10" H 8200 2200 50  0000 L CNN
+F 1 "wire" V 8150 1950 50  0000 L CNN
+F 2 "Resistor_THT:R_Axial_DIN0207_L6.3mm_D2.5mm_P7.62mm_Horizontal" V 8080 2050 50  0001 C CNN
+F 3 "~" H 8150 2050 50  0001 C CNN
+	1    8150 2050
+	-1   0    0    1
+$EndComp
 $EndSCHEMATC

Commit message: Revision 1.2.0
Parts:
- C10: value 47pF -> 100pF
Changed lines of the file:
@@
 AR Path="/5EC57429/5FC2AF22" Ref="C10"  Part="1"
 F 0 "C10" V 7950 1600 50  0000 L CNN
-F 1 "47pF" V 7950 1800 50  0000 L CNN
+F 1 "100pF" V 7950 1800 50  0000 L CNN
 F 2 "Capacitor_THT:C_Disc_D5.0mm_W2.5mm_P2.50mm" H 8050 1900 50  0001 C CNN
 F 3 "~" H 8050 1900 50  0001 C CNN
